File: hardware/BREAD_Slice.kicad_sch (KiCad schematic)
At the start: 15 parts, among them J1 Conn_01x10_Female, J2 I2C_01x04

Commit message: Initial commit
Parts:
- removed C1, C3, C4: 22uF, Capacitor_SMD:C_1206_3216Metric, symbol Device:C_Small
- removed C2: 100nF, Capacitor_SMD:C_1206_3216Metric, symbol Device:C_Small
- removed D1: WS2812B_5050, SparkFun-LED:WS2812-5050-4PIN, symbol SparkFun-LED:WS2812B_5050
- removed HS1: Heatsink_Pad, SparkFun-Fuse:Thermal Pad, symbol Mechanical:Heatsink_Pad
- removed J2: I2C_01x04, Connector_JST:JST_SH_SM04B-SRSS-TB_1x04-1MP_P1.00mm_Horizontal, symbol SparkFun-Connector:I2C_01x04
- removed L1: 4.7uH, Inductor_SMD:L_1210_3225Metric, symbol Device:L_Small
- removed U1: ~, Package_TO_SOT_SMD:TSOT-23-6, symbol SparkFun-DiscreteSemi:AP63205
- added A1, A2, A3, A4: Pololu_Breakout_A4988, Module:Pololu_Breakout-16_15.2x20.3mm, symbol Driver_Motor:Pololu_Breakout_A4988
- added C1, C2, C3: 10uF_t, OCI_UPL_FOOTPRINTS:C_2312, symbol BREAD_Slice-rescue:10uF_t-OCI_UPL_2_Capacitors-BREAD_Slice-rescue
- added D1, D2, D3, D4: 5V, Diode_SMD:D_1206_3216Metric_Pad1.42x1.75mm_HandSolder, symbol Device:D_Zener
- added J2: Screw_Terminal_01x04, TerminalBlock_TE-Connectivity:TerminalBlock_TE_282834-4_1x04_P2.54mm_Horizontal, symbol Connector:Screw_Terminal_01x04
- added J3, J4: Screw_Terminal_01x08, TerminalBlock_TE-Connectivity:TerminalBlock_TE_282834-8_1x08_P2.54mm_Horizontal, symbol Connector:Screw_Terminal_01x08
- added J5: Conn_01x03_Male, Connector_PinSocket_2.54mm:PinSocket_1x03_P2.54mm_Vertical, symbol Connector:Conn_01x03_Male
- added J6: Screw_Terminal_01x02, TerminalBlock_TE-Connectivity:TerminalBlock_TE_282834-2_1x02_P2.54mm_Horizontal, symbol Connector:Screw_Terminal_01x02
- added Logo1: Logo_Open_Hardware_Small, Symbol:OSHW-Symbol_6.7x6mm_SilkScreen, symbol Graphic:Logo_Open_Hardware_Small
- added R1, R2, R3, R4: 1k, Resistor_SMD:R_1206_3216Metric_Pad1.30x1.75mm_HandSolder, symbol Device:R
- H1, H4: footprint MountingHole:MountingHole_5mm -> MountingHole:MountingHole_3.2mm_M3_DIN965_Pad
- H2: renamed from H3; footprint MountingHole:MountingHole_5mm -> MountingHole:MountingHole_3.2mm_M3_DIN965_Pad
- H3: renamed from H2; footprint MountingHole:MountingHole_5mm -> MountingHole:MountingHole_3.2mm_M3_DIN965_Pad
- renumbered A1 to G1
Connections:
- net +12V: now also G1.30 (VIN), C1.1, J5.2 (Pin_2)
- net +5V: now also A1.2 (VDD), A2.2 (VDD), A3.2 (VDD), A4.2 (VDD), C2.1
- net GND: now also A1.1 (GND), A1.7 (GND), A2.1 (GND), A2.7 (GND), A3.1 (GND), A3.7 (GND), A4.1 (GND), A4.7 (GND), C1.2, C2.2, C3.2, D1.2 (A), D2.2 (A), D3.2 (A), D4.2 (A), J6.2 (Pin_2)
- net ST_2: now reaches G1.10 (D7)
- net ST_2: now also A2.15 (STEP)
- net DR_2: now reaches G1.11 (D8)
- net DR_2: now also A2.16 (DIR)
- net ST_3: now reaches G1.12 (D9)
- net ST_3: now also A3.15 (STEP)
- net DR_3: now reaches G1.13 (D10)
- net DR_3: now also A3.16 (DIR)
- net ST_4: now reaches G1.14 (D11)
- net ST_4: now also A4.15 (STEP)
- net DR_4: now reaches G1.15 (D12)
- net DR_4: now also A4.16 (DIR)
- net MS3: now reaches G1.16 (D13)
- net MS3: now also A1.12 (MS3), A2.12 (MS3), A3.12 (MS3), A4.12 (MS3)
- net AG_1: now reaches G1.19 (A0)
- net AG_1: now also D1.1 (K), R1.2
- net AG_2: now reaches G1.20 (A1)
- net AG_2: now also D2.1 (K), R2.2
- net AG_3: now reaches G1.21 (A2)
- net AG_3: now also D3.1 (K), R3.2
- net AG_4: now reaches G1.22 (A3)
- net AG_4: now also D4.1 (K), R4.2
- net MS1: now reaches G1.25 (A6)
- net MS1: now also A1.10 (MS1), A2.10 (MS1), A3.10 (MS1), A4.10 (MS1)
- net MS2: now reaches G1.26 (A7)
- net MS2: now also A1.11 (MS2), A2.11 (MS2), A3.11 (MS2), A4.11 (MS2)
- net DR_1: now reaches G1.9 (D6)
- net DR_1: now also A1.16 (DIR)
- net LED renamed ST_1
- net ST_1: now also A1.15 (STEP)
- new net: A1.13 (~{RESET}), A1.14 (~{SLEEP})
- new net: A2.13 (~{RESET}), A2.14 (~{SLEEP})
- new net: A3.13 (~{RESET}), A3.14 (~{SLEEP})
- new net: A4.13 (~{RESET}), A4.14 (~{SLEEP})
- new net: C3.1, J5.1 (Pin_1), J6.1 (Pin_1)
- new net 1_1A: A1.4 (1A), J3.6 (Pin_6)
- new net 1_1B: A1.3 (1B), J3.5 (Pin_5)
- new net 1_2A: A1.5 (2A), J3.7 (Pin_7)
- new net 1_2B: A1.6 (2B), J3.8 (Pin_8)
- new net 2_1A: A2.4 (1A), J3.2 (Pin_2)
- new net 2_1B: A2.3 (1B), J3.1 (Pin_1)
- new net 2_2A: A2.5 (2A), J3.3 (Pin_3)
- new net 2_2B: A2.6 (2B), J3.4 (Pin_4)
- new net 3_1A: A3.4 (1A), J4.3 (Pin_3)
- new net 3_1B: A3.3 (1B), J4.4 (Pin_4)
- new net 3_2A: A3.5 (2A), J4.2 (Pin_2)
- new net 3_2B: A3.6 (2B), J4.1 (Pin_1)
- new net 4_1A: A4.4 (1A), J4.7 (Pin_7)
- new net 4_1B: A4.3 (1B), J4.8 (Pin_8)
- new net 4_2A: A4.5 (2A), J4.6 (Pin_6)
- new net 4_2B: A4.6 (2B), J4.5 (Pin_5)
- new net A_IN1: J2.1 (Pin_1), R1.1
- new net A_IN2: J2.2 (Pin_2), R2.1
- new net A_IN3: J2.3 (Pin_3), R3.1
- new net A_IN4: J2.4 (Pin_4), R4.1
- new net M_POWER: A1.8 (VMOT), A2.8 (VMOT), A3.8 (VMOT), A4.8 (VMOT), J5.3 (Pin_3)
- no-connect marks 22 -> 10
Other:
- moved on the sheet: G1, H1, H2, H3, H4, J1
