File: hardware/BREAD_Slice.kicad_pcb (KiCad board)
At the start: 2 copper layers, 72.6 x 100 mm, 16 parts, among them J1 Conn_01x10_Female, J2 I2C_01x04

Commit message: Initial commit
Parts:
- removed C4: 22uF, Capacitor_SMD:C_1206_3216Metric
- removed HS1: Heatsink_Pad, SparkFun-Fuse:Thermal Pad
- removed L1: 4.7uH, Inductor_SMD:L_1210_3225Metric
- removed U1: ~, Package_TO_SOT_SMD:TSOT-23-6
- added A1: Pololu_Breakout_A4988, Module:Pololu_Breakout-16_15.2x20.3mm, F.Cu at (174.7, 60.4)
- added A2: Pololu_Breakout_A4988, Module:Pololu_Breakout-16_15.2x20.3mm, F.Cu at (174.7, 83.3)
- added A3: Pololu_Breakout_A4988, Module:Pololu_Breakout-16_15.2x20.3mm, F.Cu at (174.7, 106.1)
- added A4: Pololu_Breakout_A4988, Module:Pololu_Breakout-16_15.2x20.3mm, F.Cu at (174.7, 129.6)
- added D2: 5V, Diode_SMD:D_1206_3216Metric_Pad1.42x1.75mm_HandSolder, B.Cu at (146.1, 60.4)
- added D3: 5V, Diode_SMD:D_1206_3216Metric_Pad1.42x1.75mm_HandSolder, B.Cu at (139.7, 73.1)
- added D4: 5V, Diode_SMD:D_1206_3216Metric_Pad1.42x1.75mm_HandSolder, B.Cu at (146.1, 73.1)
- added J3: Screw_Terminal_01x08, TerminalBlock_TE-Connectivity:TerminalBlock_TE_282834-8_1x08_P2.54mm_Horizontal, F.Cu at (187.4, 83.9)
- added J4: Screw_Terminal_01x08, TerminalBlock_TE-Connectivity:TerminalBlock_TE_282834-8_1x08_P2.54mm_Horizontal, F.Cu at (187.4, 91.5)
- added J5: Conn_01x03_Male, Connector_PinSocket_2.54mm:PinSocket_1x03_P2.54mm_Vertical, F.Cu at (187.4, 118.8)
- added J6: Screw_Terminal_01x02, TerminalBlock_TE-Connectivity:TerminalBlock_TE_282834-2_1x02_P2.54mm_Horizontal, F.Cu at (187.4, 125.8)
- added R1: 1k, Resistor_SMD:R_1206_3216Metric_Pad1.30x1.75mm_HandSolder, B.Cu at (139.7, 54.1)
- added R2: 1k, Resistor_SMD:R_1206_3216Metric_Pad1.30x1.75mm_HandSolder, B.Cu at (146.1, 54.1)
- added R3: 1k, Resistor_SMD:R_1206_3216Metric_Pad1.30x1.75mm_HandSolder, B.Cu at (139.7, 66.8)
- added R4: 1k, Resistor_SMD:R_1206_3216Metric_Pad1.30x1.75mm_HandSolder, B.Cu at (146.1, 66.8)
- C1, C3: value 22uF -> 10uF_t; footprint Capacitor_SMD:C_1206_3216Metric -> OCI_UPL_FOOTPRINTS:C_2312
- C2: value 100nF -> 10uF_t; footprint Capacitor_SMD:C_1206_3216Metric -> OCI_UPL_FOOTPRINTS:C_2312
- D1: value WS2812B_5050 -> 5V; footprint SparkFun-LED:WS2812-5050-4PIN -> Diode_SMD:D_1206_3216Metric_Pad1.42x1.75mm_HandSolder; moved to B.Cu
- H1, H4: footprint MountingHole:MountingHole_5mm -> MountingHole:MountingHole_3.2mm_M3_DIN965_Pad
- H2: renamed from H3; footprint MountingHole:MountingHole_5mm -> MountingHole:MountingHole_3.2mm_M3_DIN965_Pad
- H3: renamed from H2; footprint MountingHole:MountingHole_5mm -> MountingHole:MountingHole_3.2mm_M3_DIN965_Pad
- J2: value I2C_01x04 -> Screw_Terminal_01x04; footprint Connector_JST:JST_SH_SM04B-SRSS-TB_1x04-1MP_P1.00mm_Horizontal -> TerminalBlock_TE-Connectivity:TerminalBlock_TE_282834-4_1x04_P2.54mm_Horizontal; moved to F.Cu
- moved J2 92.1 mm to (187.4, 52.2), turned to -90 degrees
- moved D1 82.8 mm to (139.7, 60.4), turned to 180 degrees
- moved Logo1 75.1 mm to (166.6, 135.8), turned to 0 degrees
- moved C2 70.4 mm to (126.4, 56.0), turned to 90 degrees
- moved C1 52.1 mm to (126.4, 67.4), turned to 90 degrees
- moved C3 47.4 mm to (178.5, 135.4), turned to 180 degrees
- moved G1 7.59 mm to (135.0, 100.0)
- moved J1 3.43 mm to (129.6, 78.8)
- renumbered A1 to G1
Connections:
- C1 pad 1: GND -> +12V
- C1 pad 2: +12V -> GND
- C2 pad 1: Net-(U1-SW) -> +5V
- C2 pad 2: Net-(U1-BST) -> GND
- C3 pad 1: GND -> Net-(C3-Pad1)
- C3 pad 2: +5V -> GND
- D1 pad 1: +5V -> /AG_1
- D1 pad 2: unconnected-(D1-DOUT-Pad2) -> GND
- G1 pad 1: unconnected-(A1-D1/TX-Pad1) -> Net-(G1-Pad1)
- G1 pad 10: unconnected-(A1-D7-Pad10) -> /ST_2
- G1 pad 11: unconnected-(A1-D8-Pad11) -> /DR_2
- G1 pad 12: unconnected-(A1-D9-Pad12) -> /ST_3
- G1 pad 13: unconnected-(A1-D10-Pad13) -> /DR_3
- G1 pad 14: unconnected-(A1-D11-Pad14) -> /ST_4
- G1 pad 15: unconnected-(A1-D12-Pad15) -> /DR_4
- G1 pad 16: unconnected-(A1-D13-Pad16) -> /MS3
- G1 pad 17: unconnected-(A1-3V3-Pad17) -> Net-(G1-Pad17)
- G1 pad 18: unconnected-(A1-AREF-Pad18) -> Net-(G1-Pad18)
- G1 pad 19: unconnected-(A1-A0-Pad19) -> /AG_1
- G1 pad 2: unconnected-(A1-D0/RX-Pad2) -> Net-(G1-Pad2)
- G1 pad 20: unconnected-(A1-A1-Pad20) -> /AG_2
- G1 pad 21: unconnected-(A1-A2-Pad21) -> /AG_3
- G1 pad 22: unconnected-(A1-A3-Pad22) -> /AG_4
- G1 pad 25: unconnected-(A1-A6-Pad25) -> /MS1
- G1 pad 26: unconnected-(A1-A7-Pad26) -> /MS2
- G1 pad 28: unconnected-(A1-~{RESET}-Pad28) -> Net-(G1-Pad28)
- G1 pad 3: unconnected-(A1-~{RESET}-Pad3) -> Net-(G1-Pad3)
- G1 pad 30: unconnected-(A1-VIN-Pad30) -> +12V
- G1 pad 8: /LED -> /ST_1
- G1 pad 9: unconnected-(A1-D6-Pad9) -> /DR_1
- J2 pad 1: GND -> /A_IN1
- J2 pad 2: +5V -> /A_IN2
- J2 pad 3: /I2C_DAT -> /A_IN3
- J2 pad 4: /I2C_CLK -> /A_IN4
Routing:
- net /MS1: track 0.00 -> 131.1 mm, vias 0 -> 4
- net +12V: track 46.8 -> 170.6 mm, vias 0 -> 2
- net /MS3: track 0.00 -> 105.0 mm, vias 0 -> 2
- net /M_POWER: track 0.00 -> 101.8 mm, vias 0 -> 2
- net /MS2: track 0.00 -> 98.8 mm, vias 0 -> 5
- net /AG_3: track 0.00 -> 94.9 mm, vias 0 -> 5
- net /AG_2: track 0.00 -> 86.0 mm, vias 0 -> 3
- net /DR_1: track 0.00 -> 82.2 mm, vias 0 -> 2
- net /ST_1: track 0.00 -> 81.9 mm, vias 0 -> 2
- net /AG_1: track 0.00 -> 81.2 mm, vias 0 -> 3
- net /DR_2: track 0.00 -> 66.1 mm, vias 0 -> 1
- net /ST_2: track 0.00 -> 65.6 mm, vias 0 -> 1
- net /AG_4: track 0.00 -> 58.7 mm, vias 0 -> 1
- net /A_IN3: track 0.00 -> 54.7 mm
- net /A_IN1: track 0.00 -> 53.7 mm
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- added copper zone on F.Cu, net +12V
- added copper zone on F.Cu, net +5V
Other:
- board size 72.6 x 100 mm -> 70 x 100 mm
- board text added: "+"
- board text added: "-"
- board text added: "1"
- board text added: "1A"
- board text added: "1B"
- board text added: "2"
- board text added: "2A"
- board text added: "2B"
- board text added: "3"
- board text added: "4"
- board text added: "Analog In"
- board text added: "CUSTOM"
- board text added: "CUSTOM PWR"
- board text added: "Motor 1"
- board text added: "Motor 2"
- board text added: "Motor 3"
- board text added: "Motor 4"
- board text added: "OUT"
- board text added: "STEP DRIVER 1"
- board text added: "STEP DRIVER 2"
- board text added: "STEP DRIVER 3"
- board text added: "STEP DRIVER 4"
- board text added: "Stepper Slice SLC_STEP R0 2021"
- board text removed: "12V->5V Reg"
- board text removed: "5V I2C Connector"
- board text removed: "BREAD Slice Template SLC_TEMP <version> <year>"
- board text removed: "LED"

Commit message: minor tweaks
Parts:
- added G***: LOGO, LOGO, F.Cu at (95.0, 88.0)
Other:
- board text added: "BREAD Slice Stepper Driver (SLC_STEP) Cam K Brooks rev.A [09-2024]"
- board text removed: "Stepper Slice SLC_STEP R0 2021"
